File: Comm_Bridge.kicad_pcb (KiCad board)
At the start: 2 copper layers, 66 x 55.9 mm, 98 parts, among them P1 USB_B, P2 CONN_01X03, P3 Solenoid, P4 XT60, P5 CONN_01X03, P6 CONN_01X03, U1 FT4232H, U10 ADM3251E, U11 ADM3251E, U2 93LC56BT-I/OT, U3 74HC595_CUST, U4 LM1117-XX, U5 ADC101S021, U6 NLSX4373, U7 NLSX4373, U8 ACPL-247-500E, U9 ACPL-247-500E, Y1 12MHz

Commit message: Synchronize with the subtree
Parts:
- R14: value 10k -> 12k 1%
- moved C21 3.30 mm to (173.5, 104.6)
Connections:
- U1 pad 60: Net-(U1-Pad60) -> Net-(R9-Pad1)
- U5 pad 2: Net-(C21-Pad2) -> GND
- U5 pad 3: GND -> Net-(C21-Pad2)
- U6 pad 5: GND -> VBUS
- U7 pad 5: GND -> VBUS
Routing:
- net GND: track 8.38 -> 73.3 mm, vias 2 -> 9
- net Net-(R9-Pad1): track 10.5 -> 26.7 mm
- net VBUS: track 181.5 -> 196.3 mm
- net Net-(C21-Pad2): track 18.2 -> 22.9 mm
- net Net-(R13-Pad1): track 30.1 -> 32.7 mm
- net Net-(R12-Pad1): track 28.2 -> 29.6 mm
- net Net-(R11-Pad1): track 23.4 -> 24.5 mm
- net Net-(R16-Pad1): track 47.8 -> 48.8 mm
- net Net-(U1-Pad18): track 67.5 -> 68.4 mm
- net Net-(C10-Pad1): track 22.5 -> 21.6 mm
- net Net-(U1-Pad52): track 42.0 -> 42.9 mm
- net Net-(C11-Pad1): track 27.4 -> 26.6 mm
